Commit message: update sixaxis simulation script

File: robnux_arm_sim/urdf/sixaxis_robot.urdf.xacro (robot description, xacro)
@@ -1,30 +1,38 @@
 <?xml version="1.0" ?>
 <!--
-  SixAxis_1 6-DOF serial arm URDF (Mitsubishi articulated convention)
-  Joints: JOINT_0_ACT through JOINT_5_ACT, all revolute.
-  DH parameters used in simulation scripts (Craig convention):
-    alpha = [0,   -PI/2,  0,   -PI/2,  PI/2,  -PI/2]
-    a     = [0,    0.075, 0.25,  0.03,  0,      0   ]
-    theta = [0,    PI/2,  0,     0,     0,      0   ]    (home offsets)
-    d     = [0.33, 0,     0,     0.25,  0,      0.09]
-  URDF joint origins (simplified, approximate from DH):
-    JOINT_0_ACT: xyz=(0,0,0)   Z-axis  (waist)
-    JOINT_1_ACT: xyz=(0,0,D0)  Y-axis  (shoulder pitch)
-    JOINT_2_ACT: xyz=(0,A2,0)  Y-axis  (elbow)   [arm along Y after J1 +90 offset]
-    JOINT_3_ACT: xyz=(0,A3,0)  X-axis  (forearm roll)
-    JOINT_4_ACT: xyz=(0,0,-D3) Y-axis  (wrist pitch)
-    JOINT_5_ACT: xyz=(0,0,-D5) Z-axis  (wrist roll)
+  SixAxis_1 6-DOF serial arm URDF — Craig 1989 DH convention.
+  All 6 revolute joints share axis = Z (DH convention: rotation is always Rot_z(q)).
+  Each joint <origin> encodes the fixed part of the DH transform at q=0:
+    T_fixed_i = Trans_x(a[i]) * Rot_x(alpha[i]) * Trans_z(d[i]) * Rot_z(theta_offset[i])
+  DH parameters:
+    i   alpha[i]  a[i]    d[i]   theta_offset[i]
+    0     0        0      0.330      0
+    1  -PI/2     0.075    0        PI/2
+    2     0       0.250    0         0
+    3  -PI/2     0.030   0.250      0
+    4   PI/2     0        0         0
+    5  -PI/2     0        0.090     0
+  Derived joint origins (xyz in parent frame, rpy = rotation of child frame):
+    JOINT_0_ACT: xyz=(0,0,0.33)      rpy=(0,0,0)
+    JOINT_1_ACT: xyz=(0.075,0,0)     rpy=(-PI/2, PI/2, 0)
+    JOINT_2_ACT: xyz=(0.25,0,0)      rpy=(0,0,0)
+    JOINT_3_ACT: xyz=(0.03,0.25,0)   rpy=(-PI/2,0,0)
+    JOINT_4_ACT: xyz=(0,0,0)         rpy=(PI/2,0,0)
+    JOINT_5_ACT: xyz=(0,0.09,0)      rpy=(-PI/2,0,0)
+  Home FK (q=0): EE at x=-0.265, y=0, z=0.05 — arm extends in -X direction.
+  The EE frame is at link_6 origin.
 -->
 <robot name="sixaxis_robot" xmlns:xacro="http://ros.org/wiki/xacro">
   <xacro:property name="PI"    value="3.14159265358979"/>
-  <xacro:property name="D0"   value="0.33"/>   <!-- base to shoulder height -->
-  <xacro:property name="A1"   value="0.075"/>  <!-- shoulder horizontal offset -->
-  <xacro:property name="A2"   value="0.25"/>   <!-- upper arm -->
-  <xacro:property name="A3"   value="0.03"/>   <!-- elbow geometry offset -->
-  <xacro:property name="D3"   value="0.25"/>   <!-- forearm length -->
-  <xacro:property name="D5"   value="0.09"/>   <!-- tool length -->
-  <xacro:property name="LINK_R"  value="0.035"/>
+  <!-- DH parameters -->
+  <xacro:property name="D0"   value="0.33"/>    <!-- d[0]: waist height -->
+  <xacro:property name="A1"   value="0.075"/>   <!-- a[1]: shoulder lateral offset -->
+  <xacro:property name="A2"   value="0.25"/>    <!-- a[2]: upper arm length -->
+  <xacro:property name="A3"   value="0.03"/>    <!-- a[3]: elbow geometry offset -->
+  <xacro:property name="D3"   value="0.25"/>    <!-- d[3]: forearm length -->
+  <xacro:property name="D5"   value="0.09"/>    <!-- d[5]: wrist-to-tool length -->
+  <xacro:property name="LINK_R"    value="0.030"/>
   <xacro:property name="LINK_MASS" value="2.0"/>
-  <!-- world -->
+  <!-- ── world ─────────────────────────────────────────────────── -->
   <link name="world"/>
   <joint name="world_to_base" type="fixed">
@@ -33,57 +41,69 @@
     <origin xyz="0 0 0" rpy="0 0 0"/>
   </joint>
-  <!-- base -->
+  <!-- base: visual pillar up to shoulder height D0 -->
   <link name="base_link">
     <inertial>
-      <origin xyz="0 0 0.06" rpy="0 0 0"/>
+      <origin xyz="0 0 ${D0/2}" rpy="0 0 0"/>
       <mass value="10.0"/>
       <inertia ixx="0.1" ixy="0" ixz="0" iyy="0.1" iyz="0" izz="0.05"/>
     </inertial>
     <visual>
-      <origin xyz="0 0 0.065" rpy="0 0 0"/>
-      <geometry><cylinder radius="0.08" length="0.13"/></geometry>
+      <origin xyz="0 0 ${D0/2}" rpy="0 0 0"/>
+      <geometry><cylinder radius="0.060" length="${D0}"/></geometry>
       <material name="base_grey"><color rgba="0.4 0.4 0.4 1"/></material>
     </visual>
     <collision>
-      <origin xyz="0 0 0.065" rpy="0 0 0"/>
-      <geometry><cylinder radius="0.08" length="0.13"/></geometry>
-    </collision>
-  </link>
-  <!-- ======================================================= J0: waist (revolute Z) -->
+      <origin xyz="0 0 ${D0/2}" rpy="0 0 0"/>
+      <geometry><cylinder radius="0.060" length="${D0}"/></geometry>
+    </collision>
+  </link>
+  <!-- ── J0: waist ── T_fixed_0 = Trans_z(D0) ─────────────────── -->
   <joint name="JOINT_0_ACT" type="revolute">
     <parent link="base_link"/>
     <child  link="link_1"/>
-    <origin xyz="0 0 0.13" rpy="0 0 0"/>
+    <origin xyz="0 0 ${D0}" rpy="0 0 0"/>
     <axis xyz="0 0 1"/>
     <limit lower="${-PI}" upper="${PI}" effort="200" velocity="2.09"/>
     <dynamics damping="0.5" friction="0.2"/>
   </joint>
-  <!-- trunk / column -->
+  <!-- link_1: waist hub + stub toward J1 (A1 along X of frame 0) -->
   <link name="link_1">
     <inertial>
-      <origin xyz="0 0 ${D0/2}" rpy="0 0 0"/>
-      <mass value="${LINK_MASS * 1.5}"/>
-      <inertia ixx="0.05" ixy="0" ixz="0" iyy="0.05" iyz="0" izz="0.01"/>
-    </inertial>
-    <visual>
-      <origin xyz="0 0 ${D0/2}" rpy="0 0 0"/>
-      <geometry><cylinder radius="${LINK_R}" length="${D0}"/></geometry>
+      <origin xyz="${A1/2} 0 0" rpy="0 ${PI/2} 0"/>
+      <mass value="${LINK_MASS}"/>
+      <inertia ixx="0.01" ixy="0" ixz="0" iyy="0.01" iyz="0" izz="0.005"/>
+    </inertial>
+    <!-- shoulder hub sphere -->
+    <visual>
+      <origin xyz="0 0 0" rpy="0 0 0"/>
+      <geometry><sphere radius="${LINK_R * 1.3}"/></geometry>
       <material name="blue"><color rgba="0.1 0.3 0.8 1"/></material>
     </visual>
-    <collision>
-      <origin xyz="0 0 ${D0/2}" rpy="0 0 0"/>
-      <geometry><cylinder radius="${LINK_R}" length="${D0}"/></geometry>
-    </collision>
-  </link>
-  <!-- ======================================================= J1: shoulder pitch (revolute Y) -->
+    <!-- stub cylinder from hub to J1 along X -->
+    <visual>
+      <origin xyz="${A1/2} 0 0" rpy="0 ${PI/2} 0"/>
+      <geometry><cylinder radius="${LINK_R * 0.7}" length="${A1}"/></geometry>
+      <material name="silver"><color rgba="0.7 0.7 0.8 1"/></material>
+    </visual>
+    <collision>
+      <origin xyz="${A1/2} 0 0" rpy="0 ${PI/2} 0"/>
+      <geometry><cylinder radius="${LINK_R * 0.7}" length="${A1}"/></geometry>
+    </collision>
+  </link>
+  <!-- ── J1: shoulder pitch ──────────────────────────────────────
+       T_fixed_1 = Trans_x(A1) * Rot_x(-PI/2) * Rot_z(PI/2)
+         xyz = (A1, 0, 0)
+         R   = Rot_x(-PI/2)*Rot_z(PI/2) = [[0,-1,0],[0,0,1],[-1,0,0]]
+         rpy = (-PI/2, PI/2, 0)
+  ─────────────────────────────────────────────────────────────── -->
   <joint name="JOINT_1_ACT" type="revolute">
     <parent link="link_1"/>
     <child  link="link_2"/>
-    <origin xyz="${A1} 0 ${D0}" rpy="0 0 0"/>
-    <axis xyz="0 1 0"/>
-    <limit lower="${-PI/2}" upper="${PI}" effort="150" velocity="2.09"/>
+    <origin xyz="${A1} 0 0" rpy="${-PI/2} ${PI/2} 0"/>
+    <axis xyz="0 0 1"/>
+    <limit lower="${-PI}" upper="${PI}" effort="150" velocity="2.09"/>
     <dynamics damping="0.5" friction="0.2"/>
   </joint>
-  <!-- upper arm -->
+  <!-- link_2: upper arm from J1 to J2 (A2 along X of frame 1) -->
   <link name="link_2">
     <inertial>
@@ -92,4 +112,11 @@
       <inertia ixx="0.02" ixy="0" ixz="0" iyy="0.02" iyz="0" izz="0.005"/>
     </inertial>
+    <!-- shoulder joint sphere -->
+    <visual>
+      <origin xyz="0 0 0" rpy="0 0 0"/>
+      <geometry><sphere radius="${LINK_R * 1.1}"/></geometry>
+      <material name="blue"><color rgba="0.1 0.3 0.8 1"/></material>
+    </visual>
+    <!-- upper arm cylinder along X -->
     <visual>
       <origin xyz="${A2/2} 0 0" rpy="0 ${PI/2} 0"/>
@@ -97,10 +124,4 @@
       <material name="silver"><color rgba="0.8 0.8 0.85 1"/></material>
     </visual>
-    <!-- shoulder hub -->
-    <visual>
-      <origin xyz="0 0 0" rpy="0 0 0"/>
-      <geometry><sphere radius="${LINK_R * 1.2}"/></geometry>
-      <material name="blue"><color rgba="0.1 0.3 0.8 1"/></material>
-    </visual>
     <collision>
       <origin xyz="${A2/2} 0 0" rpy="0 ${PI/2} 0"/>
@@ -108,46 +129,54 @@
     </collision>
   </link>
-  <!-- ======================================================= J2: elbow pitch (revolute Y) -->
+  <!-- ── J2: elbow ──────────────────────────────────────────────
+       T_fixed_2 = Trans_x(A2) * Rot_x(0) * Rot_z(0)
+         xyz = (A2, 0, 0),  R = I,  rpy = (0,0,0)
+  ─────────────────────────────────────────────────────────────── -->
   <joint name="JOINT_2_ACT" type="revolute">
     <parent link="link_2"/>
     <child  link="link_3"/>
     <origin xyz="${A2} 0 0" rpy="0 0 0"/>
-    <axis xyz="0 1 0"/>
-    <limit lower="${-PI}" upper="${PI/2}" effort="100" velocity="2.61"/>
+    <axis xyz="0 0 1"/>
+    <limit lower="${-PI}" upper="${PI}" effort="100" velocity="2.61"/>
     <dynamics damping="0.3" friction="0.1"/>
   </joint>
-  <!-- forearm -->
+  <!-- link_3: forearm from J2 to J3 (primarily D3 along Y, minor A3 along X) -->
   <link name="link_3">
     <inertial>
-      <origin xyz="${D3/2} 0 0" rpy="0 ${PI/2} 0"/>
+      <origin xyz="${A3/2} ${D3/2} 0" rpy="${-PI/2} 0 0"/>
       <mass value="${LINK_MASS * 0.8}"/>
       <inertia ixx="0.015" ixy="0" ixz="0" iyy="0.015" iyz="0" izz="0.004"/>
     </inertial>
-    <!-- elbow hub -->
-    <visual>
-      <origin xyz="0 0 0" rpy="0 0 0"/>
-      <geometry><sphere radius="${LINK_R * 1.1}"/></geometry>
+    <!-- elbow hub sphere -->
+    <visual>
+      <origin xyz="0 0 0" rpy="0 0 0"/>
+      <geometry><sphere radius="${LINK_R * 1.0}"/></geometry>
       <material name="blue"><color rgba="0.1 0.3 0.8 1"/></material>
     </visual>
-    <!-- forearm tube -->
-    <visual>
-      <origin xyz="${D3/2} 0 0" rpy="0 ${PI/2} 0"/>
+    <!-- forearm cylinder: center at (A3/2, D3/2, 0), along Y (rpy="-PI/2 0 0") -->
+    <visual>
+      <origin xyz="${A3/2} ${D3/2} 0" rpy="${-PI/2} 0 0"/>
       <geometry><cylinder radius="${LINK_R * 0.85}" length="${D3}"/></geometry>
       <material name="silver"><color rgba="0.8 0.8 0.85 1"/></material>
     </visual>
     <collision>
-      <origin xyz="${D3/2} 0 0" rpy="0 ${PI/2} 0"/>
+      <origin xyz="${A3/2} ${D3/2} 0" rpy="${-PI/2} 0 0"/>
       <geometry><cylinder radius="${LINK_R * 0.85}" length="${D3}"/></geometry>
     </collision>
   </link>
-  <!-- ======================================================= J3: forearm roll (revolute X) -->
+  <!-- ── J3: wrist yaw ──────────────────────────────────────────
+       T_fixed_3 = Trans_x(A3) * Rot_x(-PI/2) * Trans_z(D3)
+         Rot_x(-PI/2)*(0,0,D3) = (0, D3, 0)  →  xyz = (A3, D3, 0)
+         R = Rot_x(-PI/2),  rpy = (-PI/2, 0, 0)
+  ─────────────────────────────────────────────────────────────── -->
   <joint name="JOINT_3_ACT" type="revolute">
     <parent link="link_3"/>
     <child  link="link_4"/>
-    <origin xyz="${D3} 0 0" rpy="0 0 0"/>
-    <axis xyz="1 0 0"/>
+    <origin xyz="${A3} ${D3} 0" rpy="${-PI/2} 0 0"/>
+    <axis xyz="0 0 1"/>
     <limit lower="${-PI}" upper="${PI}" effort="60" velocity="3.14"/>
     <dynamics damping="0.2" friction="0.1"/>
   </joint>
+  <!-- link_4: wrist hub at J3/J4 -->
   <link name="link_4">
     <inertial>
@@ -166,60 +195,68 @@
     </collision>
   </link>
-  <!-- ======================================================= J4: wrist pitch (revolute Y) -->
+  <!-- ── J4: wrist pitch ────────────────────────────────────────
+       T_fixed_4 = Rot_x(PI/2),  xyz = (0,0,0),  rpy = (PI/2, 0, 0)
+  ─────────────────────────────────────────────────────────────── -->
   <joint name="JOINT_4_ACT" type="revolute">
     <parent link="link_4"/>
     <child  link="link_5"/>
-    <origin xyz="0 0 0" rpy="0 0 0"/>
-    <axis xyz="0 1 0"/>
+    <origin xyz="0 0 0" rpy="${PI/2} 0 0"/>
+    <axis xyz="0 0 1"/>
     <limit lower="${-PI * 0.75}" upper="${PI * 0.75}" effort="30" velocity="3.66"/>
     <dynamics damping="0.1" friction="0.05"/>
   </joint>
+  <!-- link_5: wrist arm from J4 to J5 (D5 along Y of frame 4) -->
   <link name="link_5">
     <inertial>
-      <origin xyz="0 0 ${-D5 * 0.4}" rpy="0 0 0"/>
+      <origin xyz="0 ${D5/2} 0" rpy="${-PI/2} 0 0"/>
       <mass value="0.3"/>
       <inertia ixx="0.001" ixy="0" ixz="0" iyy="0.001" iyz="0" izz="0.0005"/>
     </inertial>
-    <visual>
-      <origin xyz="0 0 0" rpy="0 0 0"/>
-      <geometry><sphere radius="${LINK_R * 0.8}"/></geometry>
-      <material name="blue"><color rgba="0.1 0.3 0.8 1"/></material>
-    </visual>
-    <collision>
-      <origin xyz="0 0 0" rpy="0 0 0"/>
-      <geometry><sphere radius="${LINK_R * 0.8}"/></geometry>
-    </collision>
-  </link>
-  <!-- ======================================================= J5: wrist roll (revolute X) -->
+    <!-- wrist tube along Y, from (0,0,0) to (0,D5,0) -->
+    <visual>
+      <origin xyz="0 ${D5/2} 0" rpy="${-PI/2} 0 0"/>
+      <geometry><cylinder radius="0.022" length="${D5}"/></geometry>
+      <material name="dark"><color rgba="0.25 0.25 0.25 1"/></material>
+    </visual>
+    <collision>
+      <origin xyz="0 ${D5/2} 0" rpy="${-PI/2} 0 0"/>
+      <geometry><cylinder radius="0.022" length="${D5}"/></geometry>
+    </collision>
+  </link>
+  <!-- ── J5: wrist roll ─────────────────────────────────────────
+       T_fixed_5 = Rot_x(-PI/2) * Trans_z(D5)
+         Rot_x(-PI/2)*(0,0,D5) = (0, D5, 0)  →  xyz = (0, D5, 0)
+         R = Rot_x(-PI/2),  rpy = (-PI/2, 0, 0)
+  ─────────────────────────────────────────────────────────────── -->
   <joint name="JOINT_5_ACT" type="revolute">
     <parent link="link_5"/>
     <child  link="link_6"/>
-    <origin xyz="0 0 0" rpy="0 0 0"/>
-    <axis xyz="1 0 0"/>
+    <origin xyz="0 ${D5} 0" rpy="${-PI/2} 0 0"/>
+    <axis xyz="0 0 1"/>
     <limit lower="${-PI}" upper="${PI}" effort="20" velocity="5.23"/>
     <dynamics damping="0.05" friction="0.02"/>
   </joint>
-  <!-- tool / end-effector -->
+  <!-- link_6: end-effector — TCP is at the origin of this frame -->
   <link name="link_6">
     <inertial>
-      <origin xyz="0 0 ${-D5/2}" rpy="0 0 0"/>
-      <mass value="0.15"/>
-      <inertia ixx="0.0005" ixy="0" ixz="0" iyy="0.0005" iyz="0" izz="0.0002"/>
-    </inertial>
-    <!-- wrist cylinder -->
-    <visual>
-      <origin xyz="0 0 ${-D5/2}" rpy="0 0 0"/>
-      <geometry><cylinder radius="0.02" length="${D5}"/></geometry>
-      <material name="dark"><color rgba="0.2 0.2 0.2 1"/></material>
-    </visual>
-    <!-- TCP marker -->
-    <visual>
-      <origin xyz="0 0 ${-D5}" rpy="0 0 0"/>
-      <geometry><sphere radius="0.012"/></geometry>
+      <origin xyz="0 0 0" rpy="0 0 0"/>
+      <mass value="0.10"/>
+      <inertia ixx="0.0002" ixy="0" ixz="0" iyy="0.0002" iyz="0" izz="0.0001"/>
+    </inertial>
+    <!-- TCP marker: orange sphere at EE origin -->
+    <visual>
+      <origin xyz="0 0 0" rpy="0 0 0"/>
+      <geometry><sphere radius="0.015"/></geometry>
       <material name="orange"><color rgba="1.0 0.5 0.0 1"/></material>
     </visual>
-    <collision>
-      <origin xyz="0 0 ${-D5/2}" rpy="0 0 0"/>
-      <geometry><cylinder radius="0.02" length="${D5}"/></geometry>
+    <!-- Tool Z-axis indicator: red stub along Z of EE frame -->
+    <visual>
+      <origin xyz="0 0 0.025" rpy="0 0 0"/>
+      <geometry><cylinder radius="0.006" length="0.05"/></geometry>
+      <material name="red"><color rgba="1.0 0.0 0.0 1"/></material>
+    </visual>
+    <collision>
+      <origin xyz="0 0 0" rpy="0 0 0"/>
+      <geometry><sphere radius="0.015"/></geometry>
     </collision>
   </link>
