Commit message: fix all POE FK/IK issues

File: robnux_arm_sim/urdf/poe_lite6_robot.urdf.xacro (robot description, xacro)
@@ -5,12 +5,14 @@
   POE axes at q=0 (base frame):
     J0: Z (waist)    J1: Y (shoulder, concurrent with J0)
-    J2: Z (upper arm twist)  J3: Y (forearm pitch)
+    J2: X (elbow, sideways bend)  J3: Y (forearm pitch)
     J4: Z (wrist roll)  J5: Y (wrist pitch)
   T_left translations:
     J0: (0, 0, 0.300)       J1: (0, 0, 0)   ← ZERO: J0/J1 concurrent (intersecting)
-    J2: (0, 0, 0.270)       J3: (0.280, 0, 0)  ← forearm extends along X
+    J2: (0, 0, 0.270)       J3: (0, 0, 0.280)  ← forearm extends along Z
     J4: (0, 0, 0)           J5: (0, 0, 0)   ← concurrent spherical wrist
-  Wrist pivot: (0.280, 0, 0.570)   Tool offset: (0, 0, 0.070)
-  axes[1](Y) NOT parallel to axes[2](Z) + T_left[1] norm=0 → SphericalTwoIntersecting
+  Wrist pivot: (0, 0, 0.850)   Tool offset: (0, 0, 0.070)
+  axes[1](Y) NOT parallel to axes[2](X) + T_left[1] norm=0 → SphericalTwoIntersecting
+  (J2 used to be a Z twist along the upper arm, which can never change the
+  shoulder-wrist distance: a degenerate arm whose wrist stays on a sphere.)
 -->
 <robot name="poe_lite6_robot" xmlns:xacro="http://ros.org/wiki/xacro">
@@ -18,5 +20,5 @@
   <xacro:property name="D_BASE"   value="0.300"/>  <!-- base to shoulder pivot height -->
   <xacro:property name="L_UPPER" value="0.270"/>  <!-- shoulder to upper-arm/forearm joint (Z) -->
-  <xacro:property name="L_FORE"  value="0.280"/>  <!-- forearm length (X) -->
+  <xacro:property name="L_FORE"  value="0.280"/>  <!-- forearm length (Z) -->
   <xacro:property name="D_TOOL"  value="0.070"/>  <!-- wrist to flange -->
   <xacro:property name="R"       value="0.028"/>  <!-- link tube radius -->
@@ -108,22 +110,22 @@
     </collision>
   </link>
-  <!-- J2: upper arm twist — revolute Z (NOT parallel to J1=Y → SphericalTwoIntersecting) -->
+  <!-- J2: elbow — revolute X (NOT parallel to J1=Y → SphericalTwoIntersecting) -->
   <joint name="JOINT_2_ACT" type="revolute">
     <parent link="link_2"/>
     <child  link="link_3"/>
     <origin xyz="0 0 ${L_UPPER}" rpy="0 0 0"/>
-    <axis xyz="0 0 1"/>
+    <axis xyz="1 0 0"/>
     <limit lower="${-2*PI}" upper="${2*PI}" effort="30" velocity="3.14"/>
     <dynamics damping="0.3" friction="0.1"/>
   </joint>
-  <!-- link_3: forearm along X (to wrist pivot) -->
+  <!-- link_3: forearm along Z (to wrist pivot) -->
   <link name="link_3">
     <inertial>
-      <origin xyz="${L_FORE/2} 0 0" rpy="0 ${PI/2} 0"/>
+      <origin xyz="0 0 ${L_FORE/2}" rpy="0 0 0"/>
       <mass value="${M * 0.8}"/>
       <inertia ixx="0.010" ixy="0" ixz="0" iyy="0.010" iyz="0" izz="0.002"/>
     </inertial>
     <visual>
-      <origin xyz="${L_FORE/2} 0 0" rpy="0 ${PI/2} 0"/>
+      <origin xyz="0 0 ${L_FORE/2}" rpy="0 0 0"/>
       <geometry><cylinder radius="${R*0.85}" length="${L_FORE}"/></geometry>
       <material name="lite6_white"><color rgba="0.92 0.92 0.92 1"/></material>
@@ -135,5 +137,5 @@
     </visual>
     <collision>
-      <origin xyz="${L_FORE/2} 0 0" rpy="0 ${PI/2} 0"/>
+      <origin xyz="0 0 ${L_FORE/2}" rpy="0 0 0"/>
       <geometry><cylinder radius="${R*0.85}" length="${L_FORE}"/></geometry>
     </collision>
@@ -143,5 +145,5 @@
     <parent link="link_3"/>
     <child  link="link_4"/>
-    <origin xyz="${L_FORE} 0 0" rpy="0 0 0"/>
+    <origin xyz="0 0 ${L_FORE}" rpy="0 0 0"/>
     <axis xyz="0 1 0"/>
     <limit lower="${-2.61}" upper="${2.61}" effort="30" velocity="3.14"/>
